File: rocket2-gse.kicad_sch (KiCad schematic)
At the start: 68 parts, among them J1 ARM Cortex Debug, J2 PWR0, J3 PWR1, J4 USB-C, J5 ALARM, J6 ARM, Q1 DMP3099L, Q2 DMP3099L

Commit message: Full PCB
Connections:
- net ETH_nRST is gone; now on net ETH_~{RST}: U4.3 (~{RST})
- net GND: now also U1.60 (BOOT0)
- net MCU_~{RST}: now also C10.1, R?.1
Other:
- moved on the sheet: C10, C44, R?, U1, Y?

Commit message: Revise mounting holes, remove test points
Parts:
- removed TP1: +24V, TestPoint:TestPoint_Pad_D4.0mm, symbol Connector:TestPoint
- removed TP2: +5V, TestPoint:TestPoint_Pad_D4.0mm, symbol Connector:TestPoint
- removed TP3: +3.3V, TestPoint:TestPoint_Pad_D4.0mm, symbol Connector:TestPoint
- removed TP4: GND, TestPoint:TestPoint_Pad_D4.0mm, symbol Connector:TestPoint

Commit message: Revise USB circuitry
Parts:
- added R?: 33K, Resistor_SMD:R_0402_1005Metric, symbol Device:R_Small_US
- added R?: 82K, Resistor_SMD:R_0402_1005Metric, symbol Device:R_Small_US
- added U27: USBLC6-2SC6, Package_TO_SOT_SMD:SOT-23-6, symbol Power_Protection:USBLC6-2SC6
Connections:
- net GND: now also R?.1, U27.2 (GND)
- net USB_D+: now also U27.4 (I/O2); no longer J4.A6 (D+), J4.B6 (D+)
- net USB_D-: now also U27.6 (I/O1); no longer J4.A7 (D-), J4.B7 (D-)
- net USB_VBUS renamed VBUS
- net VBUS: now also R?.2, U27.5 (VBUS); no longer U1.42 (PA9)
- new net: R?.1, R?.2, U1.42 (PA9)
- new net: J4.A7 (D-), J4.B7 (D-), U27.1 (I/O1)
- new net: J4.A6 (D+), J4.B6 (D+), U27.3 (I/O2)
Other:
- moved on the sheet: C15, C44, J1, J4, R15, R16, U4, Y?
